Commit message: First robot simulation

File: robot_module/ros2_ws/src/gesture_robot/urdf/robot.urdf.xacro (robot description, xacro)
@@ -50,10 +50,26 @@
     </inertial>
   </link>
+  <gazebo reference="left_wheel">
+      <mu1>10.0</mu1>
+      <mu2>10.0</mu2>
+      <kp>1000000.0</kp>
+      <kd>100.0</kd>
+      <minDepth>0.001</minDepth>
+      <maxVel>0.1</maxVel>
+  </gazebo>
   <joint name="left_wheel_joint" type="continuous">
     <parent link="base_link"/>
     <child link="left_wheel"/>
-    <origin xyz="0 ${base_width/2 + wheel_width/2} 0" rpy="-1.5707 0 0"/>
+    <origin xyz="0 ${base_width/2 + wheel_width/2} ${-base_height/2}" rpy="-1.5707 0 0"/>
     <axis xyz="0 0 1"/>
   </joint>
+  <gazebo reference="right_wheel">
+    <mu1>10.0</mu1>
+    <mu2>10.0</mu2>
+    <kp>1000000.0</kp>
+    <kd>100.0</kd>
+    <minDepth>0.001</minDepth>
+    <maxVel>0.1</maxVel>
+  </gazebo>
   <!-- ── Ruota destra ───────────────────────────────────────────────────── -->
   <link name="right_wheel">
@@ -77,5 +93,5 @@
     <parent link="base_link"/>
     <child link="right_wheel"/>
-    <origin xyz="0 ${-(base_width/2 + wheel_width/2)} 0" rpy="-1.5707 0 0"/>
+    <origin xyz="0 ${-(base_width/2 + wheel_width/2)} ${-base_height/2}" rpy="-1.5707 0 0"/>
     <axis xyz="0 0 1"/>
   </joint>
@@ -93,9 +109,15 @@
       </geometry>
     </collision>
-    <inertial>
-      <mass value="0.05"/>
-      <inertia ixx="0.0001" ixy="0" ixz="0" iyy="0.0001" iyz="0" izz="0.0001"/>
-    </inertial>
+  <inertial>
+    <mass value="0.001"/>
+    <inertia ixx="0.000001" ixy="0" ixz="0" iyy="0.000001" iyz="0" izz="0.000001"/>
+  </inertial>
   </link>
+  <gazebo reference="caster_wheel">
+    <mu1>0.0</mu1>
+    <mu2>0.0</mu2>
+    <kp>1000000.0</kp>
+    <kd>100.0</kd>
+</gazebo>
   <joint name="caster_joint" type="fixed">
     <parent link="base_link"/>
@@ -106,18 +128,16 @@
   <gazebo>
     <plugin name="differential_drive_controller" filename="libgazebo_ros_diff_drive.so">
-      <ros>
-        <namespace>/</namespace>
-      </ros>
+      <update_rate>30</update_rate>
       <left_joint>left_wheel_joint</left_joint>
       <right_joint>right_wheel_joint</right_joint>
-      <wheel_separation>${base_width + wheel_width}</wheel_separation>
-      <wheel_diameter>${2 * wheel_radius}</wheel_diameter>
+      <wheel_separation>0.34</wheel_separation>
+      <wheel_diameter>0.1</wheel_diameter>
       <max_wheel_torque>20</max_wheel_torque>
       <max_wheel_acceleration>1.0</max_wheel_acceleration>
-      <command_topic>cmd_vel</command_topic>
+      <command_topic>/cmd_vel</command_topic>
       <publish_odom>true</publish_odom>
       <publish_odom_tf>true</publish_odom_tf>
-      <publish_wheel_tf>true</publish_wheel_tf>
-      <odometry_topic>odom</odometry_topic>
+      <publish_wheel_tf>false</publish_wheel_tf>
+      <odometry_topic>/odom</odometry_topic>
       <odometry_frame>odom</odometry_frame>
       <robot_base_frame>base_link</robot_base_frame>
