Commit message: Fix robot head in simulation

File: install/gesture_robot/share/gesture_robot/urdf/robot.urdf.xacro (robot description, xacro)
@@ -7,11 +7,22 @@
   <xacro:property name="wheel_radius" value="0.05"/>
   <xacro:property name="wheel_width"  value="0.04"/>
-  <!-- ── Materiali ──────────────────────────────────────────────────────── -->
-  <material name="blue">
-    <color rgba="0.0 0.0 0.8 1.0"/>
+<!-- Materiale -->
+  <material name="red">
+    <color rgba="0.8 0.0 0.0 1.0"/>
   </material>
-  <material name="black">
-    <color rgba="0.0 0.0 0.0 1.0"/>
-  </material>
+  <!-- Naso frontale -->
+  <link name="front_marker">
+    <visual>
+      <geometry>
+        <box size="0.05 0.1 0.05"/>
+      </geometry>
+      <material name="red"/>
+    </visual>
+  </link>
+  <joint name="front_marker_joint" type="fixed">
+    <parent link="base_link"/>
+    <child link="front_marker"/>
+    <origin xyz="${base_length/2} 0 ${base_height/2}" rpy="0 0 0"/>
+  </joint>
   <!-- ── Base link ──────────────────────────────────────────────────────── -->
   <link name="base_link">
@@ -144,3 +155,6 @@
     </plugin>
   </gazebo>
+<gazebo reference="front_marker">
+  <material>Gazebo/Red</material>
+</gazebo>
 </robot>
